File: Arduino_ARDF/Arduino_ARDF.kicad_pcb (KiCad board)
At the start: 2 copper layers, 37 parts, among them J1 Output Mode, J2 Programming, J3 Analog 2, J4 AUX2, J5 Analog 1, J7 Analog 0, J8 AUX1, SW1 Button 1, SW2 Button 2, U1 ATmega328-P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

Commit message: Ricominciato PCB
Parts:
- JA1: moved to B.Cu
- moved R3 131.3 mm to (204.5, 62.2), turned to -90 degrees
- moved RV1 124.8 mm to (203.2, 57.1), turned to 0 degrees
- moved JP1 123.5 mm to (191.8, 69.8)
- moved C21 114.9 mm to (186.7, 52.1), turned to 180 degrees
- moved C20 114.9 mm to (188.0, 68.6), turned to -90 degrees
- moved J8 114.8 mm to (204.5, 33.0), turned to 0 degrees
- moved U1 112.6 mm to (199.4, 57.2), turned to -90 degrees
- moved D3 109.2 mm to (204.5, 74.9), turned to 90 degrees
- moved C22 108.6 mm to (177.8, 71.1)
- moved U20 108.4 mm to (181.6, 71.1), turned to 0 degrees
- moved BZ1 106.2 mm to (190.5, 43.2), turned to 180 degrees
- moved JV1 101.6 mm to (161.3, 78.7), turned to -90 degrees
- moved SW2 100.3 mm to (194.6, 51.5)
- moved SW1 94.5 mm to (194.6, 41.4)
- moved JA1 92.7 mm to (165.7, 78.7)
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Connections:
- JF3 pad 11: unconnected-(JF3-Pad11) -> CLK0
- JF3 pad 13: unconnected-(JF3-Pad13) -> CLK0
- JS1 pad 7: VIN -> +5V
Routing:
- net +5V: track 121.1 -> 178.2 mm
- net SCK: track 102.7 -> 58.2 mm
- net D3: track 5.15 -> 44.4 mm
- net A2: track 51.1 -> 16.3 mm, vias 2 -> 0
- net D2: track 5.15 -> 38.9 mm
- net LED1: track 73.3 -> 47.5 mm
- net Net-(C10-Pad1): track 4.27 -> 27.5 mm
- net VIN: track 12.6 -> 34.2 mm
- net D7: track 41.4 -> 61.6 mm
- net D5: track 62.1 -> 81.8 mm
- net A3: track 51.1 -> 32.3 mm, vias 2 -> 0
- net A1: track 43.8 -> 30.3 mm, vias 2 -> 0
- net LED2: track 52.9 -> 39.6 mm
- net SCL: track 83.3 -> 72.2 mm, vias 1 -> 0
- net SDA: track 79.0 -> 68.6 mm, vias 2 -> 0
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- added copper zone on B.Cu, net GND
- added copper zone on F.Cu, net GND
Other:
- board outline added: 69.8 x 53.3 mm
