File: Arduino_ARDF.kicad_pcb (KiCad board)
At the start: 2 copper layers, 69.8 x 53.3 mm, 37 parts, among them J1 Output Mode, J2 Programming, J3 Analog 2, J4 AUX2, J5 Analog 1, J7 Analog 0, J8 AUX1, SW1 Button 1, SW2 Button 2, U1 ATmega328-P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

Commit message: Finished PCB
Parts:
- added RV2: Potentiometer, Potentiometer_THT:Potentiometer_Vishay_T73YP_Vertical, F.Cu at (149.9, 78.7)
- renumbered D1 to L1, D2 to L2, D3 to L3
Routing:
- net A3: track 32.3 -> 78.2 mm
- net TXD: track 72.2 -> 90.5 mm, vias 1 -> 2
- net RXD: track 78.2 -> 94.3 mm, vias 1 -> 2
- net +5V: track 178.2 -> 188.6 mm
- net RST: track 65.8 -> 66.4 mm
- net D10: track 73.1 -> 73.7 mm
Other:
- board text added: "2022"
- board text added: "5V"
- board text added: "A0"
- board text added: "A1"
- board text added: "A2"
- board text added: "A3"
- board text added: "Antenna"
- board text added: "CL0"
- board text added: "CL1"
- board text added: "CL2"
- board text added: "Custom Filter Zone"
- board text added: "D10"
- board text added: "D2"
- board text added: "D3"
- board text added: "D4"
- board text added: "D5"
- board text added: "D6"
- board text added: "D7"
- board text added: "D8"
- board text added: "D9"
- board text added: "Enable 5V"
- board text added: "GND"
- board text added: "ICSP"
- board text added: "IU2FRL"
- board text added: "Input"
- board text added: "MISO"
- board text added: "MOSI"
- board text added: "No Filter/Filter"
- board text added: "Output"
- board text added: "Power"
- board text added: "Programming"
- board text added: "RST"
- board text added: "RTS"
- board text added: "RXD"
- board text added: "SCK"
- board text added: "SCL"
- board text added: "SDA"
- board text added: "SI5351"
- board text added: "SI5351 ARDF Board"
- board text added: "TXD"
- board text added: "VIN"
