File: Arduino_ARDF.kicad_sch (KiCad schematic)
At the start: 37 parts, among them J1 Output Mode, J2 Programming, J3 Analog 2, J4 AUX2, J5 Analog 1, J7 Analog 0, J8 AUX1, SW1 Button 1, SW2 Button 2, U1 ATmega328-P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

Commit message: Finished PCB
Parts:
- added RV2: Potentiometer, Potentiometer_THT:Potentiometer_Vishay_T73YP_Vertical, symbol Device:R_Potentiometer_Trim
- renumbered D1 to L1, D2 to L2, D3 to L3
Connections:
- net +5V: now also RV2.1
- net A3: now also RV2.2
- net GND: now also RV2.3
Changed lines of the file:
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@@
   (junction (at 153.67 87.63) (diameter 0) (color 0 0 0 0)
   )
+  (junction (at 201.93 149.86) (diameter 0) (color 0 0 0 0)
+  )
   (junction (at 182.88 59.69) (diameter 0) (color 0 0 0 0)
   )
@@
   )
   (junction (at 153.67 44.45) (diameter 0) (color 0 0 0 0)
+  )
+  (junction (at 201.93 160.02) (diameter 0) (color 0 0 0 0)
   )
   (junction (at 104.14 21.59) (diameter 0) (color 0 0 0 0)
@@
     (stroke (width 0) (type default) (color 0 0 0 0))
   )
+  (wire (pts (xy 220.98 160.02) (xy 201.93 160.02))
+    (stroke (width 0) (type default) (color 0 0 0 0))
+  )
   (wire (pts (xy 254 76.2) (xy 256.54 76.2))
     (stroke (width 0) (type default) (color 0 0 0 0))
@@
     (stroke (width 0) (type default) (color 0 0 0 0))
   )
+  (wire (pts (xy 201.93 149.86) (xy 220.98 149.86))
+    (stroke (width 0) (type default) (color 0 0 0 0))
+  )
   (bus (pts (xy 153.67 29.21) (xy 153.67 44.45))
     (stroke (width 0) (type default) (color 0 0 0 0))
@@
     (stroke (width 0) (type default) (color 0 0 0 0))
   )
+  (wire (pts (xy 220.98 151.13) (xy 220.98 149.86))
+    (stroke (width 0) (type default) (color 0 0 0 0))
+  )
   (wire (pts (xy 210.82 43.18) (xy 210.82 44.45))
     (stroke (width 0) (type default) (color 0 0 0 0))
@@
     (stroke (width 0) (type default) (color 0 0 0 0))
   )
+  (wire (pts (xy 224.79 154.94) (xy 226.06 154.94))
+    (stroke (width 0) (type default) (color 0 0 0 0))
+  )
   (wire (pts (xy 267.97 151.13) (xy 265.43 151.13))
     (stroke (width 0) (type default) (color 0 0 0 0))
@@
     (stroke (width 0) (type default) (color 0 0 0 0))
   )
+  (wire (pts (xy 220.98 158.75) (xy 220.98 160.02))
+    (stroke (width 0) (type default) (color 0 0 0 0))
+  )
   (wire (pts (xy 46.99 81.28) (xy 46.99 83.82))
     (stroke (width 0) (type default) (color 0 0 0 0))
@@
     (stroke (width 0) (type default) (color 0 0 0 0))
   )
+  (wire (pts (xy 201.93 148.59) (xy 201.93 149.86))
+    (stroke (width 0) (type default) (color 0 0 0 0))
+  )
   (wire (pts (xy 266.7 29.21) (xy 267.97 29.21))
     (stroke (width 0) (type default) (color 0 0 0 0))
@@
   )
   (wire (pts (xy 57.15 38.1) (xy 58.42 38.1))
+    (stroke (width 0) (type default) (color 0 0 0 0))
+  )
+  (wire (pts (xy 201.93 161.29) (xy 201.93 160.02))
     (stroke (width 0) (type default) (color 0 0 0 0))
   )
@@
     (effects (font (size 1.27 1.27)) (justify left))
     (property "Intersheet References" "${INTERSHEET_REFS}" (id 0) (at 125.5426 87.7094 0)
+      (effects (font (size 1.27 1.27)) (justify left) hide)
+    )
+  )
+  (global_label "A3" (shape input) (at 226.06 154.94 0) (fields_autoplaced)
+    (effects (font (size 1.27 1.27)) (justify left))
+    (property "Intersheet References" "${INTERSHEET_REFS}" (id 0) (at 230.7712 154.8606 0)
       (effects (font (size 1.27 1.27)) (justify left) hide)
     )
@@
   (symbol (lib_id "Device:LED") (at 167.64 114.3 180) (unit 1)
     (in_bom yes) (on_board yes) (fields_autoplaced)
-    (property "Reference" "D3" (id 0) (at 169.2275 106.68 0))
+    (property "Reference" "L3" (id 0) (at 169.2275 106.68 0))
     (property "Value" "LED" (id 1) (at 169.2275 109.22 0))
     (property "Footprint" "LED_THT:LED_D3.0mm" (id 2) (at 167.64 114.3 0)
@@
     (pin "9")
   )
+  (symbol (lib_id "Device:R_Potentiometer_Trim") (at 220.98 154.94 0) (unit 1)
+    (in_bom yes) (on_board yes)
+    (property "Reference" "RV2" (id 0) (at 218.44 154.94 0)
+      (effects (font (size 1.27 1.27)) (justify right))
+    )
+    (property "Value" "Potentiometer" (id 1) (at 234.95 160.02 0)
+      (effects (font (size 1.27 1.27)) (justify right))
+    )
+    (property "Footprint" "Potentiometer_THT:Potentiometer_Vishay_T73YP_Vertical" (id 2) (at 220.98 154.94 0)
+      (effects (font (size 1.27 1.27)) hide)
+    )
+    (property "Datasheet" "~" (id 3) (at 220.98 154.94 0)
+      (effects (font (size 1.27 1.27)) hide)
+    )
+    (pin "1")
+    (pin "2")
+    (pin "3")
+  )
   (symbol (lib_name "GND_1") (lib_id "power:GND") (at 267.97 152.4 0) (unit 1)
     (in_bom yes) (on_board yes)
@@
   )
   (symbol (lib_id "Device:R_Potentiometer_Trim") (at 201.93 154.94 0) (unit 1)
-    (in_bom yes) (on_board yes) (fields_autoplaced)
-    (property "Reference" "RV1" (id 0) (at 199.39 153.6699 0)
+    (in_bom yes) (on_board yes)
+    (property "Reference" "RV1" (id 0) (at 199.39 154.94 0)
       (effects (font (size 1.27 1.27)) (justify right))
     )
-    (property "Value" "Potentiometer" (id 1) (at 199.39 156.2099 0)
+    (property "Value" "Potentiometer" (id 1) (at 199.39 160.02 0)
       (effects (font (size 1.27 1.27)) (justify right))
     )
@@
   (symbol (lib_id "Device:LED") (at 213.36 87.63 180) (unit 1)
     (in_bom yes) (on_board yes) (fields_autoplaced)
-    (property "Reference" "D2" (id 0) (at 214.9475 80.01 0))
+    (property "Reference" "L2" (id 0) (at 214.9475 80.01 0))
     (property "Value" "LED" (id 1) (at 214.9475 82.55 0))
     (property "Footprint" "LED_THT:LED_D3.0mm" (id 2) (at 213.36 87.63 0)
@@
     (pin "1")
   )
-  (symbol (lib_id "power:+5V") (at 201.93 149.86 0) (unit 1)
-    (in_bom yes) (on_board yes) (fields_autoplaced)
-    (property "Reference" "#PWR0109" (id 0) (at 201.93 153.67 0)
+  (symbol (lib_id "power:+5V") (at 201.93 148.59 0) (unit 1)
+    (in_bom yes) (on_board yes)
+    (property "Reference" "#PWR0109" (id 0) (at 201.93 152.4 0)
       (effects (font (size 1.27 1.27)) hide)
     )
     (property "Value" "+5V" (id 1) (at 201.93 144.78 0))
-    (property "Footprint" "" (id 2) (at 201.93 149.86 0)
-      (effects (font (size 1.27 1.27)) hide)
-    )
-    (property "Datasheet" "" (id 3) (at 201.93 149.86 0)
+    (property "Footprint" "" (id 2) (at 201.93 148.59 0)
+      (effects (font (size 1.27 1.27)) hide)
+    )
+    (property "Datasheet" "" (id 3) (at 201.93 148.59 0)
       (effects (font (size 1.27 1.27)) hide)
     )
@@
     (pin "9")
   )
-  (symbol (lib_name "GND_1") (lib_id "power:GND") (at 201.93 160.02 0) (unit 1)
-    (in_bom yes) (on_board yes)
-    (property "Reference" "#PWR0108" (id 0) (at 201.93 166.37 0)
-      (effects (font (size 1.27 1.27)) hide)
-    )
-    (property "Value" "GND" (id 1) (at 205.74 161.29 0))
-    (property "Footprint" "" (id 2) (at 201.93 160.02 0)
-      (effects (font (size 1.27 1.27)) hide)
-    )
-    (property "Datasheet" "" (id 3) (at 201.93 160.02 0)
+  (symbol (lib_name "GND_1") (lib_id "power:GND") (at 201.93 161.29 0) (unit 1)
+    (in_bom yes) (on_board yes)
+    (property "Reference" "#PWR0108" (id 0) (at 201.93 167.64 0)
+      (effects (font (size 1.27 1.27)) hide)
+    )
+    (property "Value" "GND" (id 1) (at 205.74 162.56 0))
+    (property "Footprint" "" (id 2) (at 201.93 161.29 0)
+      (effects (font (size 1.27 1.27)) hide)
+    )
+    (property "Datasheet" "" (id 3) (at 201.93 161.29 0)
       (effects (font (size 1.27 1.27)) hide)
     )
@@
   (symbol (lib_id "Device:LED") (at 213.36 69.85 180) (unit 1)
     (in_bom yes) (on_board yes) (fields_autoplaced)
-    (property "Reference" "D1" (id 0) (at 214.9475 62.23 0))
+    (property "Reference" "L1" (id 0) (at 214.9475 62.23 0))
     (property "Value" "LED" (id 1) (at 214.9475 64.77 0))
     (property "Footprint" "LED_THT:LED_D3.0mm" (id 2) (at 213.36 69.85 0)
@@
       (reference "C22") (unit 1) (value "47u") (footprint "Capacitor_THT:CP_Radial_Tantal_D5.5mm_P2.50mm")
     )
-    (path "/fa27bb1a-405b-4e6b-adeb-8da937bdf19d"
-      (reference "D1") (unit 1) (value "LED") (footprint "LED_THT:LED_D3.0mm")
-    )
-    (path "/a2799286-cfb9-4343-8e3a-5c6f810527ad"
-      (reference "D2") (unit 1) (value "LED") (footprint "LED_THT:LED_D3.0mm")
-    )
-    (path "/24bddc6c-0b26-4360-8d1b-cb85b5284114"
-      (reference "D3") (unit 1) (value "LED") (footprint "LED_THT:LED_D3.0mm")
-    )
     (path "/9366b7d0-1fcb-4718-aba6-339082b6ebba"
       (reference "J1") (unit 1) (value "Output Mode") (footprint "Connector_PinHeader_2.54mm:PinHeader_1x03_P2.54mm_Vertical")
@@
       (reference "JV1") (unit 1) (value "Vin") (footprint "Connector_PinHeader_2.54mm:PinHeader_1x02_P2.54mm_Vertical")
     )
+    (path "/fa27bb1a-405b-4e6b-adeb-8da937bdf19d"
+      (reference "L1") (unit 1) (value "LED") (footprint "LED_THT:LED_D3.0mm")
+    )
+    (path "/a2799286-cfb9-4343-8e3a-5c6f810527ad"
+      (reference "L2") (unit 1) (value "LED") (footprint "LED_THT:LED_D3.0mm")
+    )
+    (path "/24bddc6c-0b26-4360-8d1b-cb85b5284114"
+      (reference "L3") (unit 1) (value "LED") (footprint "LED_THT:LED_D3.0mm")
+    )
     (path "/1b9a9b85-b0c6-4562-ac6f-dbe6fb22a155"
       (reference "R1") (unit 1) (value "470") (footprint "Resistor_THT:R_Axial_DIN0207_L6.3mm_D2.5mm_P7.62mm_Horizontal")
@@
       (reference "RV1") (unit 1) (value "Potentiometer") (footprint "Potentiometer_THT:Potentiometer_Piher_PC-16_Single_Horizontal")
     )
+    (path "/2a4c5b53-1808-4bc7-977a-c46040abafd2"
+      (reference "RV2") (unit 1) (value "Potentiometer") (footprint "Potentiometer_THT:Potentiometer_Vishay_T73YP_Vertical")
+    )
     (path "/ff64f5c9-ddc9-4c10-a08f-5c00fc1d391c"
